File: rSTM32F103VET6/rSTM32F103VET6.sch (KiCad schematic (older format))
At the start: 38 parts, among them J1 USB, J2 STLink, J3 BOOT, J4 , J5 , SW1 RESET, U1 STM32F103VET6, U2 RT9013, Y1 CSTCE8.000M, Y2 32.768K

Commit message: KiCAD Project.
Footprint fix.
Parts:
- SW1: footprint Buttons_Switches_SMD:SW_SPST_EVPBF -> .rpvM:Switch_SMD_5.2x6.4_reset
Changed lines of the file:
@@
 F 0 "SW1" H 10150 5200 50  0000 L CNN
 F 1 "RESET" H 10450 5200 50  0000 L CNN
-F 2 "Buttons_Switches_SMD:SW_SPST_EVPBF" H 10350 5250 50  0001 C CNN
+F 2 ".rpvM:Switch_SMD_5.2x6.4_reset" H 10350 5250 50  0001 C CNN
 F 3 "~" H 10350 5250 50  0001 C CNN
 	1    10350 5050
